File: 7segment.sch (KiCad schematic (older format))
At the start: 12 parts, among them J1 VCC, J2 IN_UP, J3 GND, J4 IN_DOWN, U1 LTD-2601G, U2 ATmega328P-AU

Commit message: Revision B
Parts:
- removed JP1: DIM, Jumper:SolderJumper-2_P1.3mm_Open_Pad1.0x1.5mm, symbol Jumper:SolderJumper_2_Open
- removed R1, R2: 220, Resistor_SMD:R_0805_2012Metric_Pad1.15x1.40mm_HandSolder, symbol Device:R
- added C2: 0.1uF, Capacitor_SMD:C_0805_2012Metric_Pad1.15x1.40mm_HandSolder, symbol Device:C
- added J5: AVR-ISP-6, Connector_Hirose:Hirose_DF13-06P-1.25DSA_1x06_P1.25mm_Vertical, symbol Connector:AVR-ISP-6
- added RN1, RN2: 220, Resistor_SMD:R_Array_Convex_4x0603, symbol Device:R_Pack04
Connections:
- net labels added: D0, D1, MISO, MOSI, SCK, SEG_A, SEG_B, SEG_C, SEG_D, SEG_DP, SEG_E, SEG_F, SEG_G, ~RESET
- wire segments 75 -> 72
- no-connect marks 4 -> 2

Commit message: Rev C
Parts:
- removed J5: AVR-ISP-6, Connector_Hirose:Hirose_DF13-06P-1.25DSA_1x06_P1.25mm_Vertical, symbol Connector:AVR-ISP-6
- removed JP2: DEC, Jumper:SolderJumper-2_P1.3mm_Open_Pad1.0x1.5mm, symbol Jumper:SolderJumper_2_Open
- added C3: 0.1uF, Capacitor_SMD:C_0805_2012Metric_Pad1.15x1.40mm_HandSolder, symbol Device:C
- added D1: MBR0520LT, Diode_SMD:D_SOD-123, symbol Diode:MBR0520LT
- added J5: RESET, Connector_PinHeader_2.54mm:PinHeader_1x01_P2.54mm_Vertical, symbol Connector_Generic:Conn_01x01
- added J6, J7: LATCH, Connector_PinHeader_2.54mm:PinHeader_1x01_P2.54mm_Vertical, symbol Connector_Generic:Conn_01x01
- added JP1: BIN/DEC, Connector_PinHeader_2.54mm:PinHeader_1x03_P2.54mm_Vertical, symbol Jumper:Jumper_3_Bridged12
- added JP2: LATCH MODE, Connector_PinHeader_2.54mm:PinHeader_1x03_P2.54mm_Vertical, symbol Jumper:Jumper_3_Bridged12
- added RN3: 10K, Resistor_SMD:R_Array_Convex_4x0603, symbol Device:R_Pack04
- added U3: LTD-2601G, DTLib:LTD-2601G, symbol DTLib:LTD-2601G
- RN1, RN2: value 220 -> 330
Connections:
- net labels added: D2, D3, SEL_LATCHMODE, SEL_NUMBERBASE, VIN
- wire segments 72 -> 88
- no-connect marks 2 -> 1
